File: blameless.kicad_pcb (KiCad board)
At the start: 2 copper layers, 75 x 55 mm, 60 parts, among them P1 IN, P2 VCC, P3 VEE, P4 OUT, P5 GND, Q1 BC850C, Q13 2SC2837, Q14 2SA1186, Q2 BC857, Q3 BC860C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

Commit message: Move to KiCAD 7
Other:
- net class Default removed
